Commit message: ROS1 Noetic compatibility fixes for KUKA packages

File: kuka_kr120_support/urdf/kr120r2500pro_macro.xacro (robot description, xacro)
@@ -216,4 +216,65 @@
       <origin xyz="0 0 0" rpy="0 ${radians(90)} 0"/>
     </joint>
+    <!-- TRANSMISSIONS -->
+<transmission name="${prefix}joint_a1_trans">
+  <type>transmission_interface/SimpleTransmission</type>
+  <joint name="${prefix}joint_a1">
+    <hardwareInterface>hardware_interface/PositionJointInterface</hardwareInterface>
+  </joint>
+  <actuator name="${prefix}joint_a1_motor">
+    <hardwareInterface>hardware_interface/PositionJointInterface</hardwareInterface>
+    <mechanicalReduction>1</mechanicalReduction>
+  </actuator>
+</transmission>
+<transmission name="${prefix}joint_a2_trans">
+  <type>transmission_interface/SimpleTransmission</type>
+  <joint name="${prefix}joint_a2">
+    <hardwareInterface>hardware_interface/PositionJointInterface</hardwareInterface>
+  </joint>
+  <actuator name="${prefix}joint_a2_motor">
+    <hardwareInterface>hardware_interface/PositionJointInterface</hardwareInterface>
+    <mechanicalReduction>1</mechanicalReduction>
+  </actuator>
+</transmission>
+<transmission name="${prefix}joint_a3_trans">
+  <type>transmission_interface/SimpleTransmission</type>
+  <joint name="${prefix}joint_a3">
+    <hardwareInterface>hardware_interface/PositionJointInterface</hardwareInterface>
+  </joint>
+  <actuator name="${prefix}joint_a3_motor">
+    <hardwareInterface>hardware_interface/PositionJointInterface</hardwareInterface>
+    <mechanicalReduction>1</mechanicalReduction>
+  </actuator>
+</transmission>
+<transmission name="${prefix}joint_a4_trans">
+  <type>transmission_interface/SimpleTransmission</type>
+  <joint name="${prefix}joint_a4">
+    <hardwareInterface>hardware_interface/PositionJointInterface</hardwareInterface>
+  </joint>
+  <actuator name="${prefix}joint_a4_motor">
+    <hardwareInterface>hardware_interface/PositionJointInterface</hardwareInterface>
+    <mechanicalReduction>1</mechanicalReduction>
+  </actuator>
+</transmission>
+<transmission name="${prefix}joint_a5_trans">
+  <type>transmission_interface/SimpleTransmission</type>
+  <joint name="${prefix}joint_a5">
+    <hardwareInterface>hardware_interface/PositionJointInterface</hardwareInterface>
+  </joint>
+  <actuator name="${prefix}joint_a5_motor">
+    <hardwareInterface>hardware_interface/PositionJointInterface</hardwareInterface>
+    <mechanicalReduction>1</mechanicalReduction>
+  </actuator>
+</transmission>
+<transmission name="${prefix}joint_a6_trans">
+  <type>transmission_interface/SimpleTransmission</type>
+  <joint name="${prefix}joint_a6">
+    <hardwareInterface>hardware_interface/PositionJointInterface</hardwareInterface>
+  </joint>
+  <actuator name="${prefix}joint_a6_motor">
+    <hardwareInterface>hardware_interface/PositionJointInterface</hardwareInterface>
+    <mechanicalReduction>1</mechanicalReduction>
+  </actuator>
+</transmission>
   </xacro:macro>
 </robot>

File: kuka_kr150_support/urdf/kr150_2_macro.xacro (robot description, xacro)
@@ -182,4 +182,65 @@
       <origin xyz="0 0 0" rpy="0 ${radians(90)} 0"/>
     </joint>
+    <!-- TRANSMISSIONS -->
+<transmission name="${prefix}joint_a1_trans">
+  <type>transmission_interface/SimpleTransmission</type>
+  <joint name="${prefix}joint_a1">
+    <hardwareInterface>hardware_interface/PositionJointInterface</hardwareInterface>
+  </joint>
+  <actuator name="${prefix}joint_a1_motor">
+    <hardwareInterface>hardware_interface/PositionJointInterface</hardwareInterface>
+    <mechanicalReduction>1</mechanicalReduction>
+  </actuator>
+</transmission>
+<transmission name="${prefix}joint_a2_trans">
+  <type>transmission_interface/SimpleTransmission</type>
+  <joint name="${prefix}joint_a2">
+    <hardwareInterface>hardware_interface/PositionJointInterface</hardwareInterface>
+  </joint>
+  <actuator name="${prefix}joint_a2_motor">
+    <hardwareInterface>hardware_interface/PositionJointInterface</hardwareInterface>
+    <mechanicalReduction>1</mechanicalReduction>
+  </actuator>
+</transmission>
+<transmission name="${prefix}joint_a3_trans">
+  <type>transmission_interface/SimpleTransmission</type>
+  <joint name="${prefix}joint_a3">
+    <hardwareInterface>hardware_interface/PositionJointInterface</hardwareInterface>
+  </joint>
+  <actuator name="${prefix}joint_a3_motor">
+    <hardwareInterface>hardware_interface/PositionJointInterface</hardwareInterface>
+    <mechanicalReduction>1</mechanicalReduction>
+  </actuator>
+</transmission>
+<transmission name="${prefix}joint_a4_trans">
+  <type>transmission_interface/SimpleTransmission</type>
+  <joint name="${prefix}joint_a4">
+    <hardwareInterface>hardware_interface/PositionJointInterface</hardwareInterface>
+  </joint>
+  <actuator name="${prefix}joint_a4_motor">
+    <hardwareInterface>hardware_interface/PositionJointInterface</hardwareInterface>
+    <mechanicalReduction>1</mechanicalReduction>
+  </actuator>
+</transmission>
+<transmission name="${prefix}joint_a5_trans">
+  <type>transmission_interface/SimpleTransmission</type>
+  <joint name="${prefix}joint_a5">
+    <hardwareInterface>hardware_interface/PositionJointInterface</hardwareInterface>
+  </joint>
+  <actuator name="${prefix}joint_a5_motor">
+    <hardwareInterface>hardware_interface/PositionJointInterface</hardwareInterface>
+    <mechanicalReduction>1</mechanicalReduction>
+  </actuator>
+</transmission>
+<transmission name="${prefix}joint_a6_trans">
+  <type>transmission_interface/SimpleTransmission</type>
+  <joint name="${prefix}joint_a6">
+    <hardwareInterface>hardware_interface/PositionJointInterface</hardwareInterface>
+  </joint>
+  <actuator name="${prefix}joint_a6_motor">
+    <hardwareInterface>hardware_interface/PositionJointInterface</hardwareInterface>
+    <mechanicalReduction>1</mechanicalReduction>
+  </actuator>
+</transmission>
   </xacro:macro>
 </robot>

File: kuka_kr150_support/urdf/kr150r3100_2_macro.xacro (robot description, xacro)
@@ -188,4 +188,65 @@
       <origin xyz="0 0 0" rpy="0 ${radians(90)} 0"/>
     </joint>
+    <!-- TRANSMISSIONS -->
+<transmission name="${prefix}joint_a1_trans">
+  <type>transmission_interface/SimpleTransmission</type>
+  <joint name="${prefix}joint_a1">
+    <hardwareInterface>hardware_interface/PositionJointInterface</hardwareInterface>
+  </joint>
+  <actuator name="${prefix}joint_a1_motor">
+    <hardwareInterface>hardware_interface/PositionJointInterface</hardwareInterface>
+    <mechanicalReduction>1</mechanicalReduction>
+  </actuator>
+</transmission>
+<transmission name="${prefix}joint_a2_trans">
+  <type>transmission_interface/SimpleTransmission</type>
+  <joint name="${prefix}joint_a2">
+    <hardwareInterface>hardware_interface/PositionJointInterface</hardwareInterface>
+  </joint>
+  <actuator name="${prefix}joint_a2_motor">
+    <hardwareInterface>hardware_interface/PositionJointInterface</hardwareInterface>
+    <mechanicalReduction>1</mechanicalReduction>
+  </actuator>
+</transmission>
+<transmission name="${prefix}joint_a3_trans">
+  <type>transmission_interface/SimpleTransmission</type>
+  <joint name="${prefix}joint_a3">
+    <hardwareInterface>hardware_interface/PositionJointInterface</hardwareInterface>
+  </joint>
+  <actuator name="${prefix}joint_a3_motor">
+    <hardwareInterface>hardware_interface/PositionJointInterface</hardwareInterface>
+    <mechanicalReduction>1</mechanicalReduction>
+  </actuator>
+</transmission>
+<transmission name="${prefix}joint_a4_trans">
+  <type>transmission_interface/SimpleTransmission</type>
+  <joint name="${prefix}joint_a4">
+    <hardwareInterface>hardware_interface/PositionJointInterface</hardwareInterface>
+  </joint>
+  <actuator name="${prefix}joint_a4_motor">
+    <hardwareInterface>hardware_interface/PositionJointInterface</hardwareInterface>
+    <mechanicalReduction>1</mechanicalReduction>
+  </actuator>
+</transmission>
+<transmission name="${prefix}joint_a5_trans">
+  <type>transmission_interface/SimpleTransmission</type>
+  <joint name="${prefix}joint_a5">
+    <hardwareInterface>hardware_interface/PositionJointInterface</hardwareInterface>
+  </joint>
+  <actuator name="${prefix}joint_a5_motor">
+    <hardwareInterface>hardware_interface/PositionJointInterface</hardwareInterface>
+    <mechanicalReduction>1</mechanicalReduction>
+  </actuator>
+</transmission>
+<transmission name="${prefix}joint_a6_trans">
+  <type>transmission_interface/SimpleTransmission</type>
+  <joint name="${prefix}joint_a6">
+    <hardwareInterface>hardware_interface/PositionJointInterface</hardwareInterface>
+  </joint>
+  <actuator name="${prefix}joint_a6_motor">
+    <hardwareInterface>hardware_interface/PositionJointInterface</hardwareInterface>
+    <mechanicalReduction>1</mechanicalReduction>
+  </actuator>
+</transmission>
   </xacro:macro>
 </robot>

File: kuka_kr16_support/urdf/kr16_2_macro.xacro (robot description, xacro)
@@ -217,4 +217,65 @@
       <origin xyz="0 0 0" rpy="0 ${radians(90)} 0"/>
     </joint>
+    <!-- TRANSMISSIONS -->
+<transmission name="${prefix}joint_a1_trans">
+  <type>transmission_interface/SimpleTransmission</type>
+  <joint name="${prefix}joint_a1">
+    <hardwareInterface>hardware_interface/PositionJointInterface</hardwareInterface>
+  </joint>
+  <actuator name="${prefix}joint_a1_motor">
+    <hardwareInterface>hardware_interface/PositionJointInterface</hardwareInterface>
+    <mechanicalReduction>1</mechanicalReduction>
+  </actuator>
+</transmission>
+<transmission name="${prefix}joint_a2_trans">
+  <type>transmission_interface/SimpleTransmission</type>
+  <joint name="${prefix}joint_a2">
+    <hardwareInterface>hardware_interface/PositionJointInterface</hardwareInterface>
+  </joint>
+  <actuator name="${prefix}joint_a2_motor">
+    <hardwareInterface>hardware_interface/PositionJointInterface</hardwareInterface>
+    <mechanicalReduction>1</mechanicalReduction>
+  </actuator>
+</transmission>
+<transmission name="${prefix}joint_a3_trans">
+  <type>transmission_interface/SimpleTransmission</type>
+  <joint name="${prefix}joint_a3">
+    <hardwareInterface>hardware_interface/PositionJointInterface</hardwareInterface>
+  </joint>
+  <actuator name="${prefix}joint_a3_motor">
+    <hardwareInterface>hardware_interface/PositionJointInterface</hardwareInterface>
+    <mechanicalReduction>1</mechanicalReduction>
+  </actuator>
+</transmission>
+<transmission name="${prefix}joint_a4_trans">
+  <type>transmission_interface/SimpleTransmission</type>
+  <joint name="${prefix}joint_a4">
+    <hardwareInterface>hardware_interface/PositionJointInterface</hardwareInterface>
+  </joint>
+  <actuator name="${prefix}joint_a4_motor">
+    <hardwareInterface>hardware_interface/PositionJointInterface</hardwareInterface>
+    <mechanicalReduction>1</mechanicalReduction>
+  </actuator>
+</transmission>
+<transmission name="${prefix}joint_a5_trans">
+  <type>transmission_interface/SimpleTransmission</type>
+  <joint name="${prefix}joint_a5">
+    <hardwareInterface>hardware_interface/PositionJointInterface</hardwareInterface>
+  </joint>
+  <actuator name="${prefix}joint_a5_motor">
+    <hardwareInterface>hardware_interface/PositionJointInterface</hardwareInterface>
+    <mechanicalReduction>1</mechanicalReduction>
+  </actuator>
+</transmission>
+<transmission name="${prefix}joint_a6_trans">
+  <type>transmission_interface/SimpleTransmission</type>
+  <joint name="${prefix}joint_a6">
+    <hardwareInterface>hardware_interface/PositionJointInterface</hardwareInterface>
+  </joint>
+  <actuator name="${prefix}joint_a6_motor">
+    <hardwareInterface>hardware_interface/PositionJointInterface</hardwareInterface>
+    <mechanicalReduction>1</mechanicalReduction>
+  </actuator>
+</transmission>
   </xacro:macro>
 </robot>

File: kuka_kr210_support/urdf/kr210l150_macro.xacro (robot description, xacro)
@@ -228,4 +228,65 @@
       <origin xyz="0 0 0" rpy="0 0 0"/>
     </joint>
+    <!-- TRANSMISSIONS -->
+<transmission name="${prefix}joint_a1_trans">
+  <type>transmission_interface/SimpleTransmission</type>
+  <joint name="${prefix}joint_a1">
+    <hardwareInterface>hardware_interface/PositionJointInterface</hardwareInterface>
+  </joint>
+  <actuator name="${prefix}joint_a1_motor">
+    <hardwareInterface>hardware_interface/PositionJointInterface</hardwareInterface>
+    <mechanicalReduction>1</mechanicalReduction>
+  </actuator>
+</transmission>
+<transmission name="${prefix}joint_a2_trans">
+  <type>transmission_interface/SimpleTransmission</type>
+  <joint name="${prefix}joint_a2">
+    <hardwareInterface>hardware_interface/PositionJointInterface</hardwareInterface>
+  </joint>
+  <actuator name="${prefix}joint_a2_motor">
+    <hardwareInterface>hardware_interface/PositionJointInterface</hardwareInterface>
+    <mechanicalReduction>1</mechanicalReduction>
+  </actuator>
+</transmission>
+<transmission name="${prefix}joint_a3_trans">
+  <type>transmission_interface/SimpleTransmission</type>
+  <joint name="${prefix}joint_a3">
+    <hardwareInterface>hardware_interface/PositionJointInterface</hardwareInterface>
+  </joint>
+  <actuator name="${prefix}joint_a3_motor">
+    <hardwareInterface>hardware_interface/PositionJointInterface</hardwareInterface>
+    <mechanicalReduction>1</mechanicalReduction>
+  </actuator>
+</transmission>
+<transmission name="${prefix}joint_a4_trans">
+  <type>transmission_interface/SimpleTransmission</type>
+  <joint name="${prefix}joint_a4">
+    <hardwareInterface>hardware_interface/PositionJointInterface</hardwareInterface>
+  </joint>
+  <actuator name="${prefix}joint_a4_motor">
+    <hardwareInterface>hardware_interface/PositionJointInterface</hardwareInterface>
+    <mechanicalReduction>1</mechanicalReduction>
+  </actuator>
+</transmission>
+<transmission name="${prefix}joint_a5_trans">
+  <type>transmission_interface/SimpleTransmission</type>
+  <joint name="${prefix}joint_a5">
+    <hardwareInterface>hardware_interface/PositionJointInterface</hardwareInterface>
+  </joint>
+  <actuator name="${prefix}joint_a5_motor">
+    <hardwareInterface>hardware_interface/PositionJointInterface</hardwareInterface>
+    <mechanicalReduction>1</mechanicalReduction>
+  </actuator>
+</transmission>
+<transmission name="${prefix}joint_a6_trans">
+  <type>transmission_interface/SimpleTransmission</type>
+  <joint name="${prefix}joint_a6">
+    <hardwareInterface>hardware_interface/PositionJointInterface</hardwareInterface>
+  </joint>
+  <actuator name="${prefix}joint_a6_motor">
+    <hardwareInterface>hardware_interface/PositionJointInterface</hardwareInterface>
+    <mechanicalReduction>1</mechanicalReduction>
+  </actuator>
+</transmission>
   </xacro:macro>
 </robot>

File: kuka_kr3_support/urdf/kr3r540_macro.xacro (robot description, xacro)
@@ -171,4 +171,65 @@
       <origin xyz="0 0 0" rpy="0 ${radians(90)} 0"/>
     </joint>
+    <!-- TRANSMISSIONS -->
+<transmission name="${prefix}joint_a1_trans">
+  <type>transmission_interface/SimpleTransmission</type>
+  <joint name="${prefix}joint_a1">
+    <hardwareInterface>hardware_interface/PositionJointInterface</hardwareInterface>
+  </joint>
+  <actuator name="${prefix}joint_a1_motor">
+    <hardwareInterface>hardware_interface/PositionJointInterface</hardwareInterface>
+    <mechanicalReduction>1</mechanicalReduction>
+  </actuator>
+</transmission>
+<transmission name="${prefix}joint_a2_trans">
+  <type>transmission_interface/SimpleTransmission</type>
+  <joint name="${prefix}joint_a2">
+    <hardwareInterface>hardware_interface/PositionJointInterface</hardwareInterface>
+  </joint>
+  <actuator name="${prefix}joint_a2_motor">
+    <hardwareInterface>hardware_interface/PositionJointInterface</hardwareInterface>
+    <mechanicalReduction>1</mechanicalReduction>
+  </actuator>
+</transmission>
+<transmission name="${prefix}joint_a3_trans">
+  <type>transmission_interface/SimpleTransmission</type>
+  <joint name="${prefix}joint_a3">
+    <hardwareInterface>hardware_interface/PositionJointInterface</hardwareInterface>
+  </joint>
+  <actuator name="${prefix}joint_a3_motor">
+    <hardwareInterface>hardware_interface/PositionJointInterface</hardwareInterface>
+    <mechanicalReduction>1</mechanicalReduction>
+  </actuator>
+</transmission>
+<transmission name="${prefix}joint_a4_trans">
+  <type>transmission_interface/SimpleTransmission</type>
+  <joint name="${prefix}joint_a4">
+    <hardwareInterface>hardware_interface/PositionJointInterface</hardwareInterface>
+  </joint>
+  <actuator name="${prefix}joint_a4_motor">
+    <hardwareInterface>hardware_interface/PositionJointInterface</hardwareInterface>
+    <mechanicalReduction>1</mechanicalReduction>
+  </actuator>
+</transmission>
+<transmission name="${prefix}joint_a5_trans">
+  <type>transmission_interface/SimpleTransmission</type>
+  <joint name="${prefix}joint_a5">
+    <hardwareInterface>hardware_interface/PositionJointInterface</hardwareInterface>
+  </joint>
+  <actuator name="${prefix}joint_a5_motor">
+    <hardwareInterface>hardware_interface/PositionJointInterface</hardwareInterface>
+    <mechanicalReduction>1</mechanicalReduction>
+  </actuator>
+</transmission>
+<transmission name="${prefix}joint_a6_trans">
+  <type>transmission_interface/SimpleTransmission</type>
+  <joint name="${prefix}joint_a6">
+    <hardwareInterface>hardware_interface/PositionJointInterface</hardwareInterface>
+  </joint>
+  <actuator name="${prefix}joint_a6_motor">
+    <hardwareInterface>hardware_interface/PositionJointInterface</hardwareInterface>
+    <mechanicalReduction>1</mechanicalReduction>
+  </actuator>
+</transmission>
   </xacro:macro>
 </robot>

File: kuka_kr5_support/urdf/kr5_arc_macro.xacro (robot description, xacro)
@@ -278,4 +278,65 @@
       <origin xyz="0 0 0" rpy="0 ${radians(90)} 0"/>
     </joint>
+    <!-- TRANSMISSIONS -->
+<transmission name="${prefix}joint_a1_trans">
+  <type>transmission_interface/SimpleTransmission</type>
+  <joint name="${prefix}joint_a1">
+    <hardwareInterface>hardware_interface/PositionJointInterface</hardwareInterface>
+  </joint>
+  <actuator name="${prefix}joint_a1_motor">
+    <hardwareInterface>hardware_interface/PositionJointInterface</hardwareInterface>
+    <mechanicalReduction>1</mechanicalReduction>
+  </actuator>
+</transmission>
+<transmission name="${prefix}joint_a2_trans">
+  <type>transmission_interface/SimpleTransmission</type>
+  <joint name="${prefix}joint_a2">
+    <hardwareInterface>hardware_interface/PositionJointInterface</hardwareInterface>
+  </joint>
+  <actuator name="${prefix}joint_a2_motor">
+    <hardwareInterface>hardware_interface/PositionJointInterface</hardwareInterface>
+    <mechanicalReduction>1</mechanicalReduction>
+  </actuator>
+</transmission>
+<transmission name="${prefix}joint_a3_trans">
+  <type>transmission_interface/SimpleTransmission</type>
+  <joint name="${prefix}joint_a3">
+    <hardwareInterface>hardware_interface/PositionJointInterface</hardwareInterface>
+  </joint>
+  <actuator name="${prefix}joint_a3_motor">
+    <hardwareInterface>hardware_interface/PositionJointInterface</hardwareInterface>
+    <mechanicalReduction>1</mechanicalReduction>
+  </actuator>
+</transmission>
+<transmission name="${prefix}joint_a4_trans">
+  <type>transmission_interface/SimpleTransmission</type>
+  <joint name="${prefix}joint_a4">
+    <hardwareInterface>hardware_interface/PositionJointInterface</hardwareInterface>
+  </joint>
+  <actuator name="${prefix}joint_a4_motor">
+    <hardwareInterface>hardware_interface/PositionJointInterface</hardwareInterface>
+    <mechanicalReduction>1</mechanicalReduction>
+  </actuator>
+</transmission>
+<transmission name="${prefix}joint_a5_trans">
+  <type>transmission_interface/SimpleTransmission</type>
+  <joint name="${prefix}joint_a5">
+    <hardwareInterface>hardware_interface/PositionJointInterface</hardwareInterface>
+  </joint>
+  <actuator name="${prefix}joint_a5_motor">
+    <hardwareInterface>hardware_interface/PositionJointInterface</hardwareInterface>
+    <mechanicalReduction>1</mechanicalReduction>
+  </actuator>
+</transmission>
+<transmission name="${prefix}joint_a6_trans">
+  <type>transmission_interface/SimpleTransmission</type>
+  <joint name="${prefix}joint_a6">
+    <hardwareInterface>hardware_interface/PositionJointInterface</hardwareInterface>
+  </joint>
+  <actuator name="${prefix}joint_a6_motor">
+    <hardwareInterface>hardware_interface/PositionJointInterface</hardwareInterface>
+    <mechanicalReduction>1</mechanicalReduction>
+  </actuator>
+</transmission>
   </xacro:macro>
 </robot>
