Commit message: ROS1 Noetic compatibility fixes for KUKA packages

File: kuka_kr6_support/urdf/kr6r900_2_macro.xacro (robot description, xacro)
@@ -172,4 +172,65 @@
       <origin xyz="0 0 0" rpy="0 ${radians(90)} 0"/>
     </joint>
+    <!-- TRANSMISSIONS -->
+<transmission name="${prefix}joint_a1_trans">
+  <type>transmission_interface/SimpleTransmission</type>
+  <joint name="${prefix}joint_a1">
+    <hardwareInterface>hardware_interface/PositionJointInterface</hardwareInterface>
+  </joint>
+  <actuator name="${prefix}joint_a1_motor">
+    <hardwareInterface>hardware_interface/PositionJointInterface</hardwareInterface>
+    <mechanicalReduction>1</mechanicalReduction>
+  </actuator>
+</transmission>
+<transmission name="${prefix}joint_a2_trans">
+  <type>transmission_interface/SimpleTransmission</type>
+  <joint name="${prefix}joint_a2">
+    <hardwareInterface>hardware_interface/PositionJointInterface</hardwareInterface>
+  </joint>
+  <actuator name="${prefix}joint_a2_motor">
+    <hardwareInterface>hardware_interface/PositionJointInterface</hardwareInterface>
+    <mechanicalReduction>1</mechanicalReduction>
+  </actuator>
+</transmission>
+<transmission name="${prefix}joint_a3_trans">
+  <type>transmission_interface/SimpleTransmission</type>
+  <joint name="${prefix}joint_a3">
+    <hardwareInterface>hardware_interface/PositionJointInterface</hardwareInterface>
+  </joint>
+  <actuator name="${prefix}joint_a3_motor">
+    <hardwareInterface>hardware_interface/PositionJointInterface</hardwareInterface>
+    <mechanicalReduction>1</mechanicalReduction>
+  </actuator>
+</transmission>
+<transmission name="${prefix}joint_a4_trans">
+  <type>transmission_interface/SimpleTransmission</type>
+  <joint name="${prefix}joint_a4">
+    <hardwareInterface>hardware_interface/PositionJointInterface</hardwareInterface>
+  </joint>
+  <actuator name="${prefix}joint_a4_motor">
+    <hardwareInterface>hardware_interface/PositionJointInterface</hardwareInterface>
+    <mechanicalReduction>1</mechanicalReduction>
+  </actuator>
+</transmission>
+<transmission name="${prefix}joint_a5_trans">
+  <type>transmission_interface/SimpleTransmission</type>
+  <joint name="${prefix}joint_a5">
+    <hardwareInterface>hardware_interface/PositionJointInterface</hardwareInterface>
+  </joint>
+  <actuator name="${prefix}joint_a5_motor">
+    <hardwareInterface>hardware_interface/PositionJointInterface</hardwareInterface>
+    <mechanicalReduction>1</mechanicalReduction>
+  </actuator>
+</transmission>
+<transmission name="${prefix}joint_a6_trans">
+  <type>transmission_interface/SimpleTransmission</type>
+  <joint name="${prefix}joint_a6">
+    <hardwareInterface>hardware_interface/PositionJointInterface</hardwareInterface>
+  </joint>
+  <actuator name="${prefix}joint_a6_motor">
+    <hardwareInterface>hardware_interface/PositionJointInterface</hardwareInterface>
+    <mechanicalReduction>1</mechanicalReduction>
+  </actuator>
+</transmission>
   </xacro:macro>
 </robot>

File: kuka_kr6_support/urdf/kr6r900sixx_macro.xacro (robot description, xacro)
@@ -172,4 +172,65 @@
       <origin xyz="0 0 0" rpy="0 ${radians(90)} 0"/>
     </joint>
+    <!-- TRANSMISSIONS -->
+<transmission name="${prefix}joint_a1_trans">
+  <type>transmission_interface/SimpleTransmission</type>
+  <joint name="${prefix}joint_a1">
+    <hardwareInterface>hardware_interface/PositionJointInterface</hardwareInterface>
+  </joint>
+  <actuator name="${prefix}joint_a1_motor">
+    <hardwareInterface>hardware_interface/PositionJointInterface</hardwareInterface>
+    <mechanicalReduction>1</mechanicalReduction>
+  </actuator>
+</transmission>
+<transmission name="${prefix}joint_a2_trans">
+  <type>transmission_interface/SimpleTransmission</type>
+  <joint name="${prefix}joint_a2">
+    <hardwareInterface>hardware_interface/PositionJointInterface</hardwareInterface>
+  </joint>
+  <actuator name="${prefix}joint_a2_motor">
+    <hardwareInterface>hardware_interface/PositionJointInterface</hardwareInterface>
+    <mechanicalReduction>1</mechanicalReduction>
+  </actuator>
+</transmission>
+<transmission name="${prefix}joint_a3_trans">
+  <type>transmission_interface/SimpleTransmission</type>
+  <joint name="${prefix}joint_a3">
+    <hardwareInterface>hardware_interface/PositionJointInterface</hardwareInterface>
+  </joint>
+  <actuator name="${prefix}joint_a3_motor">
+    <hardwareInterface>hardware_interface/PositionJointInterface</hardwareInterface>
+    <mechanicalReduction>1</mechanicalReduction>
+  </actuator>
+</transmission>
+<transmission name="${prefix}joint_a4_trans">
+  <type>transmission_interface/SimpleTransmission</type>
+  <joint name="${prefix}joint_a4">
+    <hardwareInterface>hardware_interface/PositionJointInterface</hardwareInterface>
+  </joint>
+  <actuator name="${prefix}joint_a4_motor">
+    <hardwareInterface>hardware_interface/PositionJointInterface</hardwareInterface>
+    <mechanicalReduction>1</mechanicalReduction>
+  </actuator>
+</transmission>
+<transmission name="${prefix}joint_a5_trans">
+  <type>transmission_interface/SimpleTransmission</type>
+  <joint name="${prefix}joint_a5">
+    <hardwareInterface>hardware_interface/PositionJointInterface</hardwareInterface>
+  </joint>
+  <actuator name="${prefix}joint_a5_motor">
+    <hardwareInterface>hardware_interface/PositionJointInterface</hardwareInterface>
+    <mechanicalReduction>1</mechanicalReduction>
+  </actuator>
+</transmission>
+<transmission name="${prefix}joint_a6_trans">
+  <type>transmission_interface/SimpleTransmission</type>
+  <joint name="${prefix}joint_a6">
+    <hardwareInterface>hardware_interface/PositionJointInterface</hardwareInterface>
+  </joint>
+  <actuator name="${prefix}joint_a6_motor">
+    <hardwareInterface>hardware_interface/PositionJointInterface</hardwareInterface>
+    <mechanicalReduction>1</mechanicalReduction>
+  </actuator>
+</transmission>
   </xacro:macro>
 </robot>

File: kuka_kr6_support/urdf/kr6r900sixx_macro_updated.xacro (robot description, xacro)
@@ -3,8 +3,8 @@
   <xacro:include filename="$(find kuka_resources)/urdf/common_constants.xacro"/>
   <xacro:include filename="$(find kuka_resources)/urdf/common_materials.xacro"/>
-  <xacro:macro name="kuka_kr6r700sixx" params="prefix">
+  <xacro:macro name="kuka_kr6r900sixx" params="prefix">
     <link name="${prefix}base_link">
       <visual>
-        <origin xyz="0 0 0" rpy="0 0 0" />
+        <origin xyz="0 0 0" rpy="0 0 0"/>
         <geometry>
           <mesh filename="package://kuka_kr6_support/meshes/kr6_agilus/visual/base_link.dae" />
@@ -13,5 +13,5 @@
       </visual>
       <collision>
-        <origin xyz="0 0 0" rpy="0 0 0" />
+        <origin xyz="0 0 0" rpy="0 0 0"/>
         <geometry>
           <mesh filename="package://kuka_kr6_support/meshes/kr6_agilus/collision/base_link.stl" />
@@ -21,5 +21,5 @@
     <link name="${prefix}link_1">
       <visual>
-        <origin xyz="0 0 0" rpy="0 0 0" />
+        <origin xyz="0 0 0" rpy="0 0 0"/>
         <geometry>
           <mesh filename="package://kuka_kr6_support/meshes/kr6_agilus/visual/link_1.dae" />
@@ -27,6 +27,17 @@
         <xacro:material_kuka_orange />
       </visual>
-      <collision>
-        <origin xyz="0 0 0" rpy="0 0 0" />
+      <inertial>
+  <origin xyz="0 0 0" rpy="0 0 0"/>
+  <mass value="2.0"/>
+  <inertia
+      ixx="0.01"
+      ixy="0.0"
+      ixz="0.0"
+      iyy="0.01"
+      iyz="0.0"
+      izz="0.01"/>
+</inertial>
+      <collision>
+        <origin xyz="0 0 0" rpy="0 0 0"/>
         <geometry>
           <mesh filename="package://kuka_kr6_support/meshes/kr6_agilus/collision/link_1.stl" />
@@ -36,14 +47,25 @@
     <link name="${prefix}link_2">
       <visual>
-        <origin xyz="0 0 0" rpy="0 0 0" />
-        <geometry>
-          <mesh filename="package://kuka_kr6_support/meshes/kr6r700sixx/visual/link_2.dae" />
-        </geometry>
-        <xacro:material_kuka_orange />
-      </visual>
-      <collision>
-        <origin xyz="0 0 0" rpy="0 0 0" />
-        <geometry>
-          <mesh filename="package://kuka_kr6_support/meshes/kr6r700sixx/collision/link_2.stl" />
+        <origin xyz="0 0 0" rpy="0 0 0"/>
+        <geometry>
+          <mesh filename="package://kuka_kr6_support/meshes/kr6r900sixx/visual/link_2.dae"/>
+        </geometry>
+        <xacro:material_kuka_orange />
+      </visual>
+      <inertial>
+  <origin xyz="0 0 0" rpy="0 0 0"/>
+  <mass value="2.0"/>
+  <inertia
+      ixx="0.01"
+      ixy="0.0"
+      ixz="0.0"
+      iyy="0.01"
+      iyz="0.0"
+      izz="0.01"/>
+</inertial>
+      <collision>
+        <origin xyz="0 0 0" rpy="0 0 0"/>
+        <geometry>
+          <mesh filename="package://kuka_kr6_support/meshes/kr6r900sixx/collision/link_2.stl" />
         </geometry>
       </collision>
@@ -51,5 +73,5 @@
     <link name="${prefix}link_3">
       <visual>
-        <origin xyz="0 0 0" rpy="0 0 0" />
+        <origin xyz="0 0 0" rpy="0 0 0"/>
         <geometry>
           <mesh filename="package://kuka_kr6_support/meshes/kr6_agilus/visual/link_3.dae" />
@@ -57,6 +79,17 @@
         <xacro:material_kuka_orange />
       </visual>
-      <collision>
-        <origin xyz="0 0 0" rpy="0 0 0" />
+      <inertial>
+  <origin xyz="0 0 0" rpy="0 0 0"/>
+  <mass value="2.0"/>
+  <inertia
+      ixx="0.01"
+      ixy="0.0"
+      ixz="0.0"
+      iyy="0.01"
+      iyz="0.0"
+      izz="0.01"/>
+</inertial>
+      <collision>
+        <origin xyz="0 0 0" rpy="0 0 0"/>
         <geometry>
           <mesh filename="package://kuka_kr6_support/meshes/kr6_agilus/collision/link_3.stl" />
@@ -66,14 +99,25 @@
     <link name="${prefix}link_4">
       <visual>
-        <origin xyz="0 0 0" rpy="0 0 0" />
-        <geometry>
-          <mesh filename="package://kuka_kr6_support/meshes/kr6r700sixx/visual/link_4.dae" />
-        </geometry>
-        <xacro:material_kuka_orange />
-      </visual>
-      <collision>
-        <origin xyz="0 0 0" rpy="0 0 0" />
-        <geometry>
-          <mesh filename="package://kuka_kr6_support/meshes/kr6r700sixx/collision/link_4.stl" />
+        <origin xyz="0 0 0" rpy="0 0 0"/>
+        <geometry>
+          <mesh filename="package://kuka_kr6_support/meshes/kr6r900sixx/visual/link_4.dae" />
+        </geometry>
+        <xacro:material_kuka_orange />
+      </visual>
+      <inertial>
+  <origin xyz="0 0 0" rpy="0 0 0"/>
+  <mass value="2.0"/>
+  <inertia
+      ixx="0.01"
+      ixy="0.0"
+      ixz="0.0"
+      iyy="0.01"
+      iyz="0.0"
+      izz="0.01"/>
+</inertial>
+      <collision>
+        <origin xyz="0 0 0" rpy="0 0 0"/>
+        <geometry>
+          <mesh filename="package://kuka_kr6_support/meshes/kr6r900sixx/collision/link_4.stl" />
         </geometry>
       </collision>
@@ -81,5 +125,5 @@
     <link name="${prefix}link_5">
       <visual>
-        <origin xyz="0 0 0" rpy="0 0 0" />
+        <origin xyz="0 0 0" rpy="0 0 0"/>
         <geometry>
           <mesh filename="package://kuka_kr6_support/meshes/kr6_agilus/visual/link_5.dae" />
@@ -87,6 +131,17 @@
         <xacro:material_kuka_orange />
       </visual>
-      <collision>
-        <origin xyz="0 0 0" rpy="0 0 0" />
+      <inertial>
+  <origin xyz="0 0 0" rpy="0 0 0"/>
+  <mass value="2.0"/>
+  <inertia
+      ixx="0.01"
+      ixy="0.0"
+      ixz="0.0"
+      iyy="0.01"
+      iyz="0.0"
+      izz="0.01"/>
+</inertial>
+      <collision>
+        <origin xyz="0 0 0" rpy="0 0 0"/>
         <geometry>
           <mesh filename="package://kuka_kr6_support/meshes/kr6_agilus/collision/link_5.stl" />
@@ -96,5 +151,5 @@
     <link name="${prefix}link_6">
       <visual>
-        <origin xyz="0 0 0" rpy="0 0 0" />
+        <origin xyz="0 0 0" rpy="0 0 0"/>
         <geometry>
           <mesh filename="package://kuka_kr6_support/meshes/kr6_agilus/visual/link_6.dae" />
@@ -102,6 +157,17 @@
         <xacro:material_kuka_pedestal />
       </visual>
-      <collision>
-        <origin xyz="0 0 0" rpy="0 0 0" />
+      <inertial>
+  <origin xyz="0 0 0" rpy="0 0 0"/>
+  <mass value="2.0"/>
+  <inertia
+      ixx="0.01"
+      ixy="0.0"
+      ixz="0.0"
+      iyy="0.01"
+      iyz="0.0"
+      izz="0.01"/>
+</inertial>
+      <collision>
+        <origin xyz="0 0 0" rpy="0 0 0"/>
         <geometry>
           <mesh filename="package://kuka_kr6_support/meshes/kr6_agilus/collision/link_6.stl" />
@@ -112,9 +178,9 @@
     <link name="${prefix}flange" />
     <joint name="${prefix}joint_a1" type="revolute">
-      <origin xyz="0 0 0.4" rpy="0 0 0"/>
+      <origin xyz="0 0 0.400" rpy="0 0 0"/>
       <parent link="${prefix}base_link"/>
       <child link="${prefix}link_1"/>
       <axis xyz="0 0 -1"/>
-      <limit lower="${radians(-170)}" upper="${radians(170)}" effort="0" velocity="${radians(360)}"/>
+      <limit effort="0" lower="${-radians(170)}" upper="${radians(170)}" velocity="${radians(360)}"/>
     </joint>
     <joint name="${prefix}joint_a2" type="revolute">
@@ -123,12 +189,12 @@
       <child link="${prefix}link_2"/>
       <axis xyz="0 1 0"/>
-      <limit lower="${radians(-190)}" upper="${radians(45)}" effort="0" velocity="${radians(300)}"/>
+      <limit effort="0" lower="${-radians(190)}" upper="${radians(45)}" velocity="${radians(300)}"/>
     </joint>
     <joint name="${prefix}joint_a3" type="revolute">
-      <origin xyz="0.315 0 0" rpy="0 0 0"/>
+      <origin xyz="0.455 0 0" rpy="0 0 0"/>
       <parent link="${prefix}link_2"/>
       <child link="${prefix}link_3"/>
       <axis xyz="0 1 0"/>
-      <limit lower="${radians(-120)}" upper="${radians(156)}" effort="0" velocity="${radians(360)}"/>
+      <limit effort="0" lower="${-radians(120)}" upper="${radians(156)}" velocity="${radians(360)}"/>
     </joint>
     <joint name="${prefix}joint_a4" type="revolute">
@@ -137,12 +203,12 @@
       <child link="${prefix}link_4"/>
       <axis xyz="-1 0 0"/>
-      <limit lower="${radians(-185)}" upper="${radians(185)}" effort="0" velocity="${radians(381)}"/>
+      <limit effort="0" lower="${-radians(185)}" upper="${radians(185)}" velocity="${radians(381)}"/>
     </joint>
     <joint name="${prefix}joint_a5" type="revolute">
-      <origin xyz="0.365 0 0" rpy="0 0 0"/>
+      <origin xyz="0.420 0 0" rpy="0 0 0"/>
       <parent link="${prefix}link_4"/>
       <child link="${prefix}link_5"/>
       <axis xyz="0 1 0"/>
-      <limit lower="${radians(-120)}" upper="${radians(120)}" effort="0" velocity="${radians(388)}"/>
+      <limit effort="0" lower="${-radians(120)}" upper="${radians(120)}" velocity="${radians(388)}"/>
     </joint>
     <joint name="${prefix}joint_a6" type="revolute">
@@ -151,5 +217,5 @@
       <child link="${prefix}link_6"/>
       <axis xyz="-1 0 0"/>
-      <limit lower="${radians(-350)}" upper="${radians(350)}" effort="0" velocity="${radians(615)}"/>
+      <limit effort="0" lower="${-radians(350)}" upper="${radians(350)}" velocity="${radians(615)}"/>
     </joint>
     <joint name="${prefix}joint_a6-flange" type="fixed">
