Commit message: fixed  kuka robot xacros

File: kuka_kr3_support/urdf/kr3r540_macro.xacro (robot description, xacro)
@@ -11,4 +11,15 @@
         <xacro:material_kuka_pedestal />
       </visual>
+      <inertial>
+  <origin xyz="0 0 0" rpy="0 0 0"/>
+  <mass value="10"/>
+  <inertia
+      ixx="0.10"
+      iyy="0.10"
+      izz="0.10"
+      ixy="0"
+      ixz="0"
+      iyz="0"/>
+</inertial>
       <collision>
         <origin xyz="0 0 0" rpy="0 0 0" />
@@ -26,4 +37,15 @@
         <xacro:material_kuka_ral_pure_white />
       </visual>
+      <inertial>
+  <origin xyz="0 0 0" rpy="0 0 0"/>
+  <mass value="6"/>
+  <inertia
+      ixx="0.06"
+      iyy="0.06"
+      izz="0.06"
+      ixy="0"
+      ixz="0"
+      iyz="0"/>
+</inertial>
       <collision>
         <origin xyz="0 0 0" rpy="0 0 0" />
@@ -41,4 +63,15 @@
         <xacro:material_kuka_ral_pure_white />
       </visual>
+      <inertial>
+  <origin xyz="0 0 0" rpy="0 0 0"/>
+  <mass value="4"/>
+  <inertia
+      ixx="0.04"
+      iyy="0.04"
+      izz="0.04"
+      ixy="0"
+      ixz="0"
+      iyz="0"/>
+</inertial>
       <collision>
         <origin xyz="0 0 0" rpy="0 0 0" />
@@ -56,4 +89,15 @@
         <xacro:material_kuka_ral_pure_white />
       </visual>
+      <inertial>
+  <origin xyz="0 0 0" rpy="0 0 0"/>
+  <mass value="3"/>
+  <inertia
+      ixx="0.03"
+      iyy="0.03"
+      izz="0.03"
+      ixy="0"
+      ixz="0"
+      iyz="0"/>
+</inertial>
       <collision>
         <origin xyz="0 0 0" rpy="0 0 0" />
@@ -71,4 +115,15 @@
         <xacro:material_kuka_ral_pure_white />
       </visual>
+      <inertial>
+  <origin xyz="0 0 0" rpy="0 0 0"/>
+  <mass value="1.5"/>
+  <inertia
+      ixx="0.015"
+      iyy="0.015"
+      izz="0.015"
+      ixy="0"
+      ixz="0"
+      iyz="0"/>
+</inertial>
       <collision>
         <origin xyz="0 0 0" rpy="0 0 0" />
@@ -86,4 +141,15 @@
         <xacro:material_kuka_ral_pure_white />
       </visual>
+      <inertial>
+  <origin xyz="0 0 0" rpy="0 0 0"/>
+  <mass value="1.0"/>
+  <inertia
+      ixx="0.01"
+      iyy="0.01"
+      izz="0.01"
+      ixy="0"
+      ixz="0"
+      iyz="0"/>
+</inertial>
       <collision>
         <origin xyz="0 0 0" rpy="0 0 0" />
@@ -101,4 +167,15 @@
         <xacro:material_kuka_pedestal />
       </visual>
+      <inertial>
+  <origin xyz="0 0 0" rpy="0 0 0"/>
+  <mass value="0.5"/>
+  <inertia
+      ixx="0.005"
+      iyy="0.005"
+      izz="0.005"
+      ixy="0"
+      ixz="0"
+      iyz="0"/>
+</inertial>
       <collision>
         <origin xyz="0 0 0" rpy="0 0 0" />
@@ -115,5 +192,5 @@
       <child link="${prefix}link_1"/>
       <axis xyz="0 0 -1"/>
-      <limit lower="${radians(-170)}" upper="${radians(170)}" effort="0" velocity="${radians(530)}"/>
+      <limit lower="${radians(-170)}" upper="${radians(170)}" effort="100" velocity="${radians(530)}"/>
     </joint>
     <joint name="${prefix}joint_a2" type="revolute">
@@ -122,5 +199,5 @@
       <child link="${prefix}link_2"/>
       <axis xyz="0 1 0"/>
-      <limit lower="${radians(-170)}" upper="${radians(50)}" effort="0" velocity="${radians(529)}"/>
+      <limit lower="${radians(-170)}" upper="${radians(50)}" effort="100" velocity="${radians(529)}"/>
     </joint>
     <joint name="${prefix}joint_a3" type="revolute">
@@ -129,5 +206,5 @@
       <child link="${prefix}link_3"/>
       <axis xyz="0 1 0"/>
-      <limit lower="${radians(-110)}" upper="${radians(155)}" effort="0" velocity="${radians(538)}"/>
+      <limit lower="${radians(-110)}" upper="${radians(155)}" effort="80" velocity="${radians(538)}"/>
     </joint>
     <joint name="${prefix}joint_a4" type="revolute">
@@ -136,5 +213,5 @@
       <child link="${prefix}link_4"/>
       <axis xyz="-1 0 0"/>
-      <limit lower="${radians(-175)}" upper="${radians(175)}" effort="0" velocity="${radians(600)}"/>
+      <limit lower="${radians(-175)}" upper="${radians(175)}" effort="30" velocity="${radians(600)}"/>
     </joint>
     <joint name="${prefix}joint_a5" type="revolute">
@@ -143,5 +220,5 @@
       <child link="${prefix}link_5"/>
       <axis xyz="0 1 0"/>
-      <limit lower="${radians(-120)}" upper="${radians(120)}" effort="0" velocity="${radians(600)}"/>
+      <limit lower="${radians(-120)}" upper="${radians(120)}" effort="30" velocity="${radians(600)}"/>
     </joint>
     <joint name="${prefix}joint_a6" type="revolute">
@@ -150,5 +227,5 @@
       <child link="${prefix}link_6"/>
       <axis xyz="-1 0 0"/>
-      <limit lower="${radians(-350)}" upper="${radians(350)}" effort="0" velocity="${radians(800)}"/>
+      <limit lower="${radians(-350)}" upper="${radians(350)}" effort="15" velocity="${radians(800)}"/>
     </joint>
     <joint name="${prefix}joint_a6-tool0" type="fixed">

File: kuka_kr3_support/urdf/kr3r540_macro_updated.xacro (robot description, xacro)
@@ -1,13 +1,11 @@
 <?xml version="1.0"?>
 <robot xmlns:xacro="http://wiki.ros.org/xacro">
-  <xacro:macro name="kuka_kr150r3100_2" params="prefix">
-    <xacro:include filename="$(find kuka_resources)/urdf/common_materials.xacro"/>
-    <!-- LINKS -->
-    <!-- base link -->
+  <xacro:include filename="$(find kuka_resources)/urdf/common_materials.xacro"/>
+  <xacro:macro name="kuka_kr3r540" params="prefix">
     <link name="${prefix}base_link">
       <visual>
-        <origin rpy="0 0 0" xyz="0 0 0"/>
-        <geometry>
-          <mesh filename="package://kuka_kr150_support/meshes/kr150r3100_2/visual/base_link.stl" />
+        <origin xyz="0 0 0" rpy="0 0 0" />
+        <geometry>
+          <mesh filename="package://kuka_kr3_support/meshes/kr3r540/visual/base_link.stl" />
         </geometry>
         <xacro:material_kuka_pedestal />
@@ -15,233 +13,226 @@
       <inertial>
   <origin xyz="0 0 0" rpy="0 0 0"/>
-  <mass value="350"/>
-  <inertia
-      ixx="15.0"
-      ixy="0"
-      ixz="0"
-      iyy="15.0"
-      iyz="0"
-      izz="15.0"/>
-</inertial>
-      <collision>
-        <origin rpy="0 0 0" xyz="0 0 0"/>
-        <geometry>
-          <mesh filename="package://kuka_kr150_support/meshes/kr150r3100_2/collision/base_link.stl" />
-        </geometry>
-      </collision>
-    </link>
-    <!-- link 1 (A1) -->
+  <mass value="10"/>
+  <inertia
+      ixx="0.10"
+      iyy="0.10"
+      izz="0.10"
+      ixy="0"
+      ixz="0"
+      iyz="0"/>
+</inertial>
+      <collision>
+        <origin xyz="0 0 0" rpy="0 0 0" />
+        <geometry>
+          <mesh filename="package://kuka_kr3_support/meshes/kr3r540/collision/base_link.stl" />
+        </geometry>
+      </collision>
+    </link>
     <link name="${prefix}link_1">
       <visual>
-        <origin xyz="0 0 0" rpy="0 0 0"/>
-        <geometry>
-          <mesh filename="package://kuka_kr150_support/meshes/kr150r3100_2/visual/link_1.stl" />
-        </geometry>
-        <xacro:material_kuka_orange />
-      </visual>
-      <inertial>
-  <origin xyz="0 0 0" rpy="0 0 0"/>
-  <mass value="180"/>
-  <inertia
-      ixx="8.0"
-      ixy="0"
-      ixz="0"
-      iyy="8.0"
-      iyz="0"
-      izz="8.0"/>
-</inertial>
-      <collision>
-        <origin xyz="0 0 0" rpy="0 0 0"/>
-        <geometry>
-          <mesh filename="package://kuka_kr150_support/meshes/kr150r3100_2/collision/link_1.stl" />
-        </geometry>
-      </collision>
-    </link>
-    <!-- link 2 -->
+        <origin xyz="0 0 0" rpy="0 0 0" />
+        <geometry>
+          <mesh filename="package://kuka_kr3_support/meshes/kr3r540/visual/link_1.stl" />
+        </geometry>
+        <xacro:material_kuka_ral_pure_white />
+      </visual>
+      <inertial>
+  <origin xyz="0 0 0" rpy="0 0 0"/>
+  <mass value="6"/>
+  <inertia
+      ixx="0.06"
+      iyy="0.06"
+      izz="0.06"
+      ixy="0"
+      ixz="0"
+      iyz="0"/>
+</inertial>
+      <collision>
+        <origin xyz="0 0 0" rpy="0 0 0" />
+        <geometry>
+          <mesh filename="package://kuka_kr3_support/meshes/kr3r540/collision/link_1.stl" />
+        </geometry>
+      </collision>
+    </link>
     <link name="${prefix}link_2">
       <visual>
-        <origin xyz="0 0 0" rpy="0 0 0"/>
-        <geometry>
-          <mesh filename="package://kuka_kr150_support/meshes/kr150r3100_2/visual/link_2.stl"/>
-        </geometry>
-        <xacro:material_kuka_orange />
-      </visual>
-      <inertial>
-  <origin xyz="0 0 0" rpy="0 0 0"/>
-  <mass value="140"/>
-  <inertia
-      ixx="6.0"
-      ixy="0"
-      ixz="0"
-      iyy="6.0"
-      iyz="0"
-      izz="6.0"/>
-</inertial>
-      <collision>
-        <origin xyz="0 0 0" rpy="0 0 0"/>
-        <geometry>
-          <mesh filename="package://kuka_kr150_support/meshes/kr150r3100_2/collision/link_2.stl"  />
-        </geometry>
-      </collision>
-    </link>
-    <!-- link 3 -->
+        <origin xyz="0 0 0" rpy="0 0 0" />
+        <geometry>
+          <mesh filename="package://kuka_kr3_support/meshes/kr3r540/visual/link_2.stl" />
+        </geometry>
+        <xacro:material_kuka_ral_pure_white />
+      </visual>
+      <inertial>
+  <origin xyz="0 0 0" rpy="0 0 0"/>
+  <mass value="4"/>
+  <inertia
+      ixx="0.04"
+      iyy="0.04"
+      izz="0.04"
+      ixy="0"
+      ixz="0"
+      iyz="0"/>
+</inertial>
+      <collision>
+        <origin xyz="0 0 0" rpy="0 0 0" />
+        <geometry>
+          <mesh filename="package://kuka_kr3_support/meshes/kr3r540/collision/link_2.stl" />
+        </geometry>
+      </collision>
+    </link>
     <link name="${prefix}link_3">
       <visual>
-        <origin xyz="0 0 0" rpy="0 0 0"/>
-        <geometry>
-          <mesh filename="package://kuka_kr150_support/meshes/kr150r3100_2/visual/link_3.stl" />
-        </geometry>
-        <xacro:material_kuka_orange />
-      </visual>
-      <inertial>
-  <origin xyz="0 0 0" rpy="0 0 0"/>
-  <mass value="100"/>
-  <inertia
-      ixx="4.5"
-      ixy="0"
-      ixz="0"
-      iyy="4.5"
-      iyz="0"
-      izz="4.5"/>
-</inertial>
-      <collision>
-        <origin xyz="0 0 0" rpy="0 0 0"/>
-        <geometry>
-          <mesh filename="package://kuka_kr150_support/meshes/kr150r3100_2/collision/link_3.stl"  />
-        </geometry>
-      </collision>
-    </link>
-    <!-- link 4 -->
+        <origin xyz="0 0 0" rpy="0 0 0" />
+        <geometry>
+          <mesh filename="package://kuka_kr3_support/meshes/kr3r540/visual/link_3.stl" />
+        </geometry>
+        <xacro:material_kuka_ral_pure_white />
+      </visual>
+      <inertial>
+  <origin xyz="0 0 0" rpy="0 0 0"/>
+  <mass value="3"/>
+  <inertia
+      ixx="0.03"
+      iyy="0.03"
+      izz="0.03"
+      ixy="0"
+      ixz="0"
+      iyz="0"/>
+</inertial>
+      <collision>
+        <origin xyz="0 0 0" rpy="0 0 0" />
+        <geometry>
+          <mesh filename="package://kuka_kr3_support/meshes/kr3r540/collision/link_3.stl" />
+        </geometry>
+      </collision>
+    </link>
     <link name="${prefix}link_4">
       <visual>
-        <origin xyz="0 0 0" rpy="0 0 0"/>
-        <geometry>
-          <mesh filename="package://kuka_kr150_support/meshes/kr150r3100_2/visual/link_4.stl" />
-        </geometry>
-        <xacro:material_kuka_orange />
-      </visual>
-      <inertial>
-  <origin xyz="0 0 0" rpy="0 0 0"/>
-  <mass value="40"/>
-  <inertia
-      ixx="2.0"
-      ixy="0"
-      ixz="0"
-      iyy="2.0"
-      iyz="0"
-      izz="2.0"/>
-</inertial>
-      <collision>
-        <origin xyz="0 0 0" rpy="0 0 0"/>
-        <geometry>
-          <mesh filename="package://kuka_kr150_support/meshes/kr150r3100_2/collision/link_4.stl"  />
-        </geometry>
-      </collision>
-    </link>
-    <!-- link 5 -->
+        <origin xyz="0 0 0" rpy="0 0 0" />
+        <geometry>
+          <mesh filename="package://kuka_kr3_support/meshes/kr3r540/visual/link_4.stl" />
+        </geometry>
+        <xacro:material_kuka_ral_pure_white />
+      </visual>
+      <inertial>
+  <origin xyz="0 0 0" rpy="0 0 0"/>
+  <mass value="1.5"/>
+  <inertia
+      ixx="0.015"
+      iyy="0.015"
+      izz="0.015"
+      ixy="0"
+      ixz="0"
+      iyz="0"/>
+</inertial>
+      <collision>
+        <origin xyz="0 0 0" rpy="0 0 0" />
+        <geometry>
+          <mesh filename="package://kuka_kr3_support/meshes/kr3r540/collision/link_4.stl" />
+        </geometry>
+      </collision>
+    </link>
     <link name="${prefix}link_5">
       <visual>
-        <origin xyz="0 0 0" rpy="0 0 0"/>
-        <geometry>
-          <mesh filename="package://kuka_kr150_support/meshes/kr150r3100_2/visual/link_5.stl" />
-        </geometry>
-        <xacro:material_kuka_orange />
-      </visual>
-      <inertial>
-  <origin xyz="0 0 0" rpy="0 0 0"/>
-  <mass value="18"/>
-  <inertia
-      ixx="1.0"
-      ixy="0"
-      ixz="0"
-      iyy="1.0"
-      iyz="0"
-      izz="1.0"/>
-</inertial>
-      <collision>
-        <origin xyz="0 0 0" rpy="0 0 0"/>
-        <geometry>
-          <mesh filename="package://kuka_kr150_support/meshes/kr150r3100_2/collision/link_5.stl" />
-        </geometry>
-      </collision>
-    </link>
-    <!-- link 6 -->
+        <origin xyz="0 0 0" rpy="0 0 0" />
+        <geometry>
+          <mesh filename="package://kuka_kr3_support/meshes/kr3r540/visual/link_5.stl" />
+        </geometry>
+        <xacro:material_kuka_ral_pure_white />
+      </visual>
+      <inertial>
+  <origin xyz="0 0 0" rpy="0 0 0"/>
+  <mass value="1.0"/>
+  <inertia
+      ixx="0.01"
+      iyy="0.01"
+      izz="0.01"
+      ixy="0"
+      ixz="0"
+      iyz="0"/>
+</inertial>
+      <collision>
+        <origin xyz="0 0 0" rpy="0 0 0" />
+        <geometry>
+          <mesh filename="package://kuka_kr3_support/meshes/kr3r540/collision/link_5.stl" />
+        </geometry>
+      </collision>
+    </link>
     <link name="${prefix}link_6">
       <visual>
-        <origin xyz="0 0 0" rpy="0 0 0"/>
-        <geometry>
-          <mesh filename="package://kuka_kr150_support/meshes/kr150r3100_2/visual/link_6.stl" />
-        </geometry>
-        <xacro:material_kuka_orange />
-      </visual>
-      <inertial>
-  <origin xyz="0 0 0" rpy="0 0 0"/>
-  <mass value="8"/>
-  <inertia
-      ixx="0.4"
-      ixy="0"
-      ixz="0"
-      iyy="0.4"
-      iyz="0"
-      izz="0.4"/>
-</inertial>
-      <collision>
-        <origin xyz="0 0 0" rpy="0 0 0"/>
-        <geometry>
-          <mesh filename="package://kuka_kr150_support/meshes/kr150r3100_2/collision/link_6.stl" />
-        </geometry>
-      </collision>
-    </link>
-    <!-- END LINKS -->
-    <!-- JOINTS -->
-    <!-- joint 1 (A1) -->
+        <origin xyz="0 0 0" rpy="0 0 0" />
+        <geometry>
+          <mesh filename="package://kuka_kr3_support/meshes/kr3r540/visual/link_6.stl" />
+        </geometry>
+        <xacro:material_kuka_pedestal />
+      </visual>
+      <inertial>
+  <origin xyz="0 0 0" rpy="0 0 0"/>
+  <mass value="0.5"/>
+  <inertia
+      ixx="0.005"
+      iyy="0.005"
+      izz="0.005"
+      ixy="0"
+      ixz="0"
+      iyz="0"/>
+</inertial>
+      <collision>
+        <origin xyz="0 0 0" rpy="0 0 0" />
+        <geometry>
+          <mesh filename="package://kuka_kr3_support/meshes/kr3r540/collision/link_6.stl" />
+        </geometry>
+      </collision>
+    </link>
+    <!-- Following REP199, this frame shall be use to attach EEF or other equipment -->
+    <link name="${prefix}flange" />
     <joint name="${prefix}joint_a1" type="revolute">
-      <origin xyz="0 0 0.645" rpy="0 0 0"/>
+      <origin xyz="0 0 0.345" rpy="0 0 0"/>
       <parent link="${prefix}base_link"/>
       <child link="${prefix}link_1"/>
       <axis xyz="0 0 -1"/>
-      <limit effort="1800" lower="${radians(-185)}" upper="${radians(185)}" velocity="${radians(105)}"/>
-    </joint>
-    <!-- joint 2 (A2) -->
+      <limit lower="${radians(-170)}" upper="${radians(170)}" effort="100" velocity="${radians(530)}"/>
+    </joint>
     <joint name="${prefix}joint_a2" type="revolute">
-      <origin xyz="0.33 0 0" rpy="0 0 0"/>
+      <origin xyz="0.020 0 0" rpy="0 0 0"/>
       <parent link="${prefix}link_1"/>
       <child link="${prefix}link_2"/>
       <axis xyz="0 1 0"/>
-      <limit effort="1800" lower="${radians(-140)}" upper="${radians(-5)}" velocity="${radians(107)}"/>
-    </joint>
-    <!-- joint 3 (A3) -->
+      <limit lower="${radians(-170)}" upper="${radians(50)}" effort="100" velocity="${radians(529)}"/>
+    </joint>
     <joint name="${prefix}joint_a3" type="revolute">
-      <origin xyz="1.350 0 0" rpy="0 0 0"/>
+      <origin xyz="0.260 0 0" rpy="0 0 0"/>
       <parent link="${prefix}link_2"/>
       <child link="${prefix}link_3"/>
       <axis xyz="0 1 0"/>
-      <limit effort="1500" lower="${radians(-120)}" upper="${radians(168)}" velocity="${radians(114)}"/>
-    </joint>
-    <!-- joint 4 (A4) -->
+      <limit lower="${radians(-110)}" upper="${radians(155)}" effort="80" velocity="${radians(538)}"/>
+    </joint>
     <joint name="${prefix}joint_a4" type="revolute">
-      <origin xyz="1.420 0 0.115" rpy="0 0 0"/>
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
File: kuka_kr5_support/urdf/kr5_arc_macro_updated.xacro (robot description, xacro)
@@ -215,5 +215,5 @@
       <child link="${prefix}link_1"/>
       <axis xyz="0 0 1"/>
-      <limit effort="0" lower="${radians(-155)}" upper="${radians(155)}" velocity="${radians(154)}"/>
+      <limit effort="150" lower="${radians(-155)}" upper="${radians(155)}" velocity="${radians(154)}"/>
     </joint>
     <!-- joint 2 (A2) -->
@@ -223,5 +223,5 @@
       <child link="${prefix}link_2"/>
       <axis xyz="0 0 1"/>
-      <limit effort="0" lower="${radians(-180)}" upper="${radians(65)}" velocity="${radians(154)}"/>
+      <limit effort="150" lower="${radians(-180)}" upper="${radians(65)}" velocity="${radians(154)}"/>
     </joint>
     <!-- joint 3 (A3) -->
@@ -231,5 +231,5 @@
       <child link="${prefix}link_3"/>
       <axis xyz="0 0 1"/>
-      <limit effort="0" lower="${radians(-15)}" upper="${radians(158)}" velocity="${radians(228)}"/>
+      <limit effort="120" lower="${radians(-15)}" upper="${radians(158)}" velocity="${radians(228)}"/>
     </joint>
     <!-- joint 4 (A4) -->
@@ -239,5 +239,5 @@
       <child link="${prefix}link_4"/>
       <axis xyz="0 0 1"/>
-      <limit effort="0" lower="${radians(-350)}" upper="${radians(350)}" velocity="${radians(343)}"/>
+      <limit effort="40" lower="${radians(-350)}" upper="${radians(350)}" velocity="${radians(343)}"/>
     </joint>
     <!-- joint 5 (A5) -->
@@ -247,5 +247,5 @@
       <child link="${prefix}link_5"/>
       <axis xyz="0 0 1"/>
-      <limit effort="0" lower="${radians(-130)}" upper="${radians(130)}" velocity="${radians(384)}"/>
+      <limit effort="40" lower="${radians(-130)}" upper="${radians(130)}" velocity="${radians(384)}"/>
     </joint>
     <!-- joint 6 (A6) -->
@@ -255,5 +255,5 @@
       <child link="${prefix}link_6"/>
       <axis xyz="0 0 1"/>
-      <limit effort="0" lower="${radians(-350)}" upper="${radians(350)}" velocity="${radians(721)}"/>
+      <limit effort="20" lower="${radians(-350)}" upper="${radians(350)}" velocity="${radians(721)}"/>
     </joint>
     <!-- tool frame - fixed frame -->
